File: Quadsense.sch (KiCad schematic (older format))
At the start: 120 parts, among them IC1 BME280, IC2 MIC5205, IC3 ADC_LTC2497, IC4 BME280, IC5 ADA4528-2, IC6 ADA4528-2, IC7 ADA4528-2, IC8 MCP6034, IC9 LP5907, P3 CONN_6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

Commit message: Schematics cleanup
Other:
- note added: "1.8V"
- note added: "Biased sensors: Choose R14/R15 for bias voltage,\npopulate R20/R22 or R21/R23 for pos/neg bias.\nUnbiased sensors: Populate R20/R23, DNP R14/R15/C23."
- note added: "ISB connectors"
- note removed: "Note: 4V and A4V are actually 4.11V. Both low noise."
- note removed: "Sensor conn"
- moved on the sheet: C1, C10, C12, C13, C14, C15, C16, C2, C4, C40, C41, C42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
