File: Quadsense.kicad_pcb (KiCad board)
At the start: 2 copper layers, 90 x 100 mm, 120 parts, among them IC1 BME280, IC2 MIC5205, IC3 ADC_LTC2497, IC4 BME280, IC5 ADA4528-2, IC6 ADA4528-2, IC7 ADA4528-2, IC8 MCP6034, IC9 LP5907, P3 CONN_6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

Commit message: Changed version on silkscreen
Other:
- board text added: "OpenAir Quadsense twin V1.0 Made with Love in Cologne by Press Every Key"
- board text removed: "OpenAir Quadsense V1.1 Made with Love in Cologne by Press Every Key"
Changed lines of the file:
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@@
   )
   (setup
-    (last_trace_width 0.4)
+    (last_trace_width 0.25)
     (user_trace_width 0.2)
     (user_trace_width 0.25)
@@
       (xy -1.530848 3.031431)) (layer B.SilkS) (width 0.01))
   )
-  (gr_text "OpenAir Quadsense V1.1\nMade with Love in Cologne\nby Press Every Key" (at 151.8 129) (layer B.SilkS)
+  (gr_text "OpenAir Quadsense twin V1.0\nMade with Love in Cologne\nby Press Every Key" (at 151.8 129) (layer B.SilkS)
     (effects (font (size 1.5 1.5) (thickness 0.3)) (justify left mirror))
   )
@@
   (gr_line (start 190 50) (end 190 150) (layer Edge.Cuts) (width 0.15))
   (gr_line (start 100 50) (end 190 50) (layer Edge.Cuts) (width 0.15))
-  (via (at 148.8 105.3) (size 0.6) (drill 0.3) (layers F.Cu B.Cu) (net 2))
-  (via (at 168.1 90) (size 0.6) (drill 0.3) (layers F.Cu B.Cu) (net 2))
-  (via (at 168.3 110.2) (size 0.6) (drill 0.3) (layers F.Cu B.Cu) (net 2))
-  (via (at 169 107) (size 0.6) (drill 0.3) (layers F.Cu B.Cu) (net 2))
-  (via (at 169.8 93) (size 0.6) (drill 0.3) (layers F.Cu B.Cu) (net 2))
-  (via (at 175 78) (size 0.6) (drill 0.3) (layers F.Cu B.Cu) (net 2))
-  (via (at 175 91) (size 0.6) (drill 0.3) (layers F.Cu B.Cu) (net 2))
-  (via (at 175 104) (size 0.6) (drill 0.3) (layers F.Cu B.Cu) (net 2))
-  (via (at 175 109) (size 0.6) (drill 0.3) (layers F.Cu B.Cu) (net 2))
-  (via (at 145 140) (size 0.6) (drill 0.3) (layers F.Cu B.Cu) (net 2))
-  (via (at 102.2 82.2) (size 0.6) (drill 0.3) (layers F.Cu B.Cu) (net 2))
-  (via (at 145 53) (size 0.6) (drill 0.3) (layers F.Cu B.Cu) (net 2))
   (segment (start 141.825 68.73) (end 140.69363 68.73) (width 0.6) (layer B.Cu) (net 1) (status 10))
   (segment (start 140.69363 68.73) (end 140.31363 68.35) (width 0.6) (layer B.Cu) (net 1))
@@
   (segment (start 152.3 71.295002) (end 152.345001 71.250001) (width 0.6) (layer F.Cu) (net 1))
   (segment (start 152.3 73.8) (end 152.3 71.295002) (width 0.6) (layer F.Cu) (net 1))
+  (via (at 148.8 105.3) (size 0.6) (drill 0.3) (layers F.Cu B.Cu) (net 2))
+  (via (at 168.1 90) (size 0.6) (drill 0.3) (layers F.Cu B.Cu) (net 2))
+  (via (at 168.3 110.2) (size 0.6) (drill 0.3) (layers F.Cu B.Cu) (net 2))
+  (via (at 169 107) (size 0.6) (drill 0.3) (layers F.Cu B.Cu) (net 2))
+  (via (at 169.8 93) (size 0.6) (drill 0.3) (layers F.Cu B.Cu) (net 2))
+  (via (at 175 78) (size 0.6) (drill 0.3) (layers F.Cu B.Cu) (net 2))
+  (via (at 175 91) (size 0.6) (drill 0.3) (layers F.Cu B.Cu) (net 2))
+  (via (at 175 104) (size 0.6) (drill 0.3) (layers F.Cu B.Cu) (net 2))
+  (via (at 175 109) (size 0.6) (drill 0.3) (layers F.Cu B.Cu) (net 2))
+  (via (at 145 140) (size 0.6) (drill 0.3) (layers F.Cu B.Cu) (net 2))
+  (via (at 102.2 82.2) (size 0.6) (drill 0.3) (layers F.Cu B.Cu) (net 2))
+  (via (at 145 53) (size 0.6) (drill 0.3) (layers F.Cu B.Cu) (net 2))
   (segment (start 126.869998 115.9) (end 127.1 115.9) (width 0.25) (layer F.Cu) (net 2))
   (via (at 127.1 115.9) (size 0.6) (drill 0.3) (layers F.Cu B.Cu) (net 2))
